File: Scheme/DANI-PROJECT.sch (EAGLE design)
At the start: 29 parts, among them T1 2N2222, T2 2N2222

Commit message: simplified circuit
Parts:
- removed OK1, OK2, OK3, OK4: 4N25, optocoupler:4N37
- removed R1, R3, R5, R7: 4k7, resistor:R-EU_0207/7
- removed R2, R4, R6, R8: 10k, resistor:R-EU_0207/7
- removed S1, S2, S3, S4: (no value), con-ptr500:AK500/2-H
- added AC: (no value), con-ptr500:AK500/2-H
- added D3, D4: SFH482, led:SFH482
- added HKLP1: HKLPM01, HKLPM01:HKLPM01
- RELE: device con-ptr500:AK500/2-H -> con-ptr500:AK500/3-H
Connections:
- removed net N$10: R3.2, S2-2.KL
- removed net N$11: R5.1, S3-2.KL
- removed net N$12: OK3.A, S3-1.KL
- removed net N$13: OK4.C, R7.2
- removed net N$14: OK4.A, S4-1.KL
- removed net N$15: R7.1, S4-2.KL
- removed net N$16: OK4.COL, R8.1, U$1.D8
- removed net N$25: -.B, R10.2, R12.2, R13.1, R2.2, R4.2, R6.2, R8.2, U$1.VIN
- removed net N$3: OK1.A, S1-1.KL
- removed net N$4: OK1.COL, R2.1, U$1.D0
- removed net N$5: OK2.C, R3.1
- removed net N$6: OK3.C, R5.2
- removed net N$7: OK2.A, S2-1.KL
- removed net N$8: OK2.COL, R4.1, U$1.D1
- removed net N$9: OK3.COL, R6.1, U$1.D2
- new net N$23: -.B, HKLP1.+VO, R10.2, R12.2, R13.1, RELE-1.KL, U$1.VIN
- net N$1: now also AC-2.KL, HKLP1.AC2; no longer OK1.C, R1.1
- net N$18: now also D4.C
- net N$2: now also AC-1.KL, HKLP1.AC1; no longer R1.2, S1-2.KL
- net N$21: now also D3.A
- net N$22: now also D3.C
- net N$24: now also D4.A
- net N$28: now also HKLP1.-VO; no longer OK1.EMI, OK2.EMI, OK3.EMI, OK4.EMI
- net N$31: now also RELE-3.KL; no longer RELE-1.KL
Other:
- moved on the sheet: RELE-1, RELE-2
